File: nrf52-mesh/nrf52-mesh/nrfmodule.sch (KiCad schematic (older format))
At the start: 2 parts

Commit message: next portion
Parts:
- added J?: Conn_02x05_Odd_Even, symbol Connector_Generic:Conn_02x05_Odd_Even
Connections:
- net GND: now also J?.3 (Pin_3), J?.5 (Pin_5), J?.9 (Pin_9)
- net SWDCLK: now also J?.4 (Pin_4)
- net SWDIO: now also J?.2 (Pin_2)
- no-connect marks 0 -> 5
Changed lines of the file:
@@
 $Descr A4 11693 8268
 encoding utf-8
-Sheet 3 7
+Sheet 3 8
 Title ""
 Date ""
@@
 Text GLabel 5650 2500 2    50   Input ~ 0
 SWDIO
+$Comp
+L Connector_Generic:Conn_02x05_Odd_Even J?
+U 1 1 5E56ADA4
+P 7150 3750
+F 0 "J?" H 7200 4167 50  0000 C CNN
+F 1 "Conn_02x05_Odd_Even" H 7200 4076 50  0000 C CNN
+F 2 "" H 7150 3750 50  0001 C CNN
+F 3 "~" H 7150 3750 50  0001 C CNN
+	1    7150 3750
+	1    0    0    -1
+$EndComp
+Wire Wire Line
+	8050 3650 7450 3650
+Text GLabel 8050 3650 2    50   Input ~ 0
+SWDCLK
+Text GLabel 7750 3550 2    50   Input ~ 0
+SWDIO
+Wire Wire Line
+	7450 3550 7750 3550
+$Comp
+L power:GND #PWR?
+U 1 1 5E56D12B
+P 6650 4200
+F 0 "#PWR?" H 6650 3950 50  0001 C CNN
+F 1 "GND" H 6655 4027 50  0000 C CNN
+F 2 "" H 6650 4200 50  0001 C CNN
+F 3 "" H 6650 4200 50  0001 C CNN
+	1    6650 4200
+	1    0    0    -1
+$EndComp
+Wire Wire Line
+	6950 3650 6650 3650
+Wire Wire Line
+	6650 3650 6650 3750
+Wire Wire Line
+	6950 3750 6650 3750
+Connection ~ 6650 3750
+Wire Wire Line
+	6650 3750 6650 3950
+Wire Wire Line
+	6950 3950 6650 3950
+Connection ~ 6650 3950
+Wire Wire Line
+	6650 3950 6650 4200
+NoConn ~ 6950 3850
+NoConn ~ 7450 3950
+NoConn ~ 7450 3850
+NoConn ~ 7450 3750
+NoConn ~ 6950 3550
 $EndSCHEMATC

Commit message: CP2102N + MAX1555 + FAN5341 + TPS560200 + TLV62568
Parts:
- J1: renamed from J?; footprint (none) -> Connector_PinSocket_1.27mm:PinSocket_2x05_P1.27mm_Vertical
- gave numbers to parts that had none: 2
Connections:
- net io4: now reaches U5.10 (SIO_16)
- net io6: now reaches U5.11 (SIO_14)
- net LED1: now reaches U5.2 (SIO_24)
- net io5: now reaches U5.29 (SIO_15)
- net CAP1: now reaches U5.3 (SIO_23)
- net io3: now reaches U5.30 (SIO_17)
- net io1: now reaches U5.31 (SIO_19)
- net CHARGE: now reaches U5.32 (SIO_31/AIN7)
- net usbtx: now reaches U5.33 (SIO_30/AIN6)
- net usbrx: now reaches U5.34 (SIO_29/AIN5)
- net LEDREGEN: now reaches U5.35 (SIO_28/AIN4)
- net LED4: now reaches U5.36 (SIO_27)
- net LED3: now reaches U5.37 (SIO_26)
- net LED2: now reaches U5.38 (SIO_25)
- net CAP2: now reaches U5.4 (SIO_22)
- net CAP3: now reaches U5.7 (SIO_21)
- net CAP4: now reaches U5.8 (SIO_20)
- net io2: now reaches U5.9 (SIO_18)
- no-connect marks 5 -> 19
Changed lines of the file:
@@
 P 4350 1650
 AR Path="/5E4FC51D" Ref="#PWR?"  Part="1"
-AR Path="/5E4EF39F/5E4FC51D" Ref="#PWR?"  Part="1"
-F 0 "#PWR?" H 4350 1500 50  0001 C CNN
+AR Path="/5E4EF39F/5E4FC51D" Ref="#PWR018"  Part="1"
+F 0 "#PWR018" H 4350 1500 50  0001 C CNN
 F 1 "+3V3" H 4365 1823 50  0000 C CNN
 F 2 "" H 4350 1650 50  0001 C CNN
@@
 P 4400 4600
 AR Path="/5E4FC523" Ref="#PWR?"  Part="1"
-AR Path="/5E4EF39F/5E4FC523" Ref="#PWR?"  Part="1"
-F 0 "#PWR?" H 4400 4350 50  0001 C CNN
+AR Path="/5E4EF39F/5E4FC523" Ref="#PWR019"  Part="1"
+F 0 "#PWR019" H 4400 4350 50  0001 C CNN
 F 1 "GND" H 4405 4427 50  0000 C CNN
 F 2 "" H 4400 4600 50  0001 C CNN
@@
 P 4350 3300
 AR Path="/5E4FC536" Ref="U?"  Part="1"
-AR Path="/5E4EF39F/5E4FC536" Ref="U?"  Part="1"
-F 0 "U?" H 4350 4581 50  0000 C CNN
+AR Path="/5E4EF39F/5E4FC536" Ref="U5"  Part="1"
+F 0 "U5" H 4350 4581 50  0000 C CNN
 F 1 "BL652" H 4350 4490 50  0000 C CNN
 F 2 "RF_Module:Laird_BL652" H 4350 2100 50  0001 C CNN
@@
 $EndComp
 $Comp
-L power:GND #PWR?
+L power:GND #PWR022
 U 1 1 5E50C770
 P 8150 2300
-F 0 "#PWR?" H 8150 2050 50  0001 C CNN
+F 0 "#PWR022" H 8150 2050 50  0001 C CNN
 F 1 "GND" H 8155 2127 50  0000 C CNN
 F 2 "" H 8150 2300 50  0001 C CNN
@@
 	8100 1700 8100 1900
 $Comp
-L power:+3V3 #PWR?
+L power:+3V3 #PWR021
 U 1 1 5E50C77E
 P 8100 1700
-F 0 "#PWR?" H 8100 1550 50  0001 C CNN
+F 0 "#PWR021" H 8100 1550 50  0001 C CNN
 F 1 "+3V3" H 8115 1873 50  0000 C CNN
 F 2 "" H 8100 1700 50  0001 C CNN
@@
 $EndComp
 $Comp
-L Connector:Conn_01x04_Male J?
+L Connector:Conn_01x04_Male J2
 U 1 1 5E50C784
 P 8450 2100
-F 0 "J?" H 8422 1982 50  0000 R CNN
+F 0 "J2" H 8422 1982 50  0000 R CNN
 F 1 "Conn_01x04_Male" H 8422 2073 50  0000 R CNN
 F 2 "Connector_PinHeader_2.54mm:PinHeader_1x04_P2.54mm_Vertical" H 8450 2100 50  0001 C CNN
@@
 SWDIO
 $Comp
-L Connector_Generic:Conn_02x05_Odd_Even J?
+L Connector_Generic:Conn_02x05_Odd_Even J1
 U 1 1 5E56ADA4
 P 7150 3750
-F 0 "J?" H 7200 4167 50  0000 C CNN
+F 0 "J1" H 7200 4167 50  0000 C CNN
 F 1 "Conn_02x05_Odd_Even" H 7200 4076 50  0000 C CNN
-F 2 "" H 7150 3750 50  0001 C CNN
+F 2 "Connector_PinSocket_1.27mm:PinSocket_2x05_P1.27mm_Vertical" H 7150 3750 50  0001 C CNN
 F 3 "~" H 7150 3750 50  0001 C CNN
 	1    7150 3750
@@
 	7450 3550 7750 3550
 $Comp
-L power:GND #PWR?
+L power:GND #PWR020
 U 1 1 5E56D12B
 P 6650 4200
-F 0 "#PWR?" H 6650 3950 50  0001 C CNN
+F 0 "#PWR020" H 6650 3950 50  0001 C CNN
 F 1 "GND" H 6655 4027 50  0000 C CNN
 F 2 "" H 6650 4200 50  0001 C CNN
@@
 NoConn ~ 7450 3750
 NoConn ~ 6950 3550
+Text GLabel 5350 2800 2    50   Input ~ 0
+CHARGE
+Text GLabel 5350 3000 2    50   Input ~ 0
+usbrx
+Text GLabel 5350 2900 2    50   Input ~ 0
+usbtx
+Text GLabel 5350 3100 2    50   Input ~ 0
+LEDREGEN
+Text GLabel 5350 3500 2    50   Input ~ 0
+LED1
+Text GLabel 5350 3400 2    50   Input ~ 0
+LED2
+Text GLabel 5350 3300 2    50   Input ~ 0
+LED3
+Text GLabel 5350 3200 2    50   Input ~ 0
+LED4
+Text GLabel 5350 3600 2    50   Input ~ 0
+CAP1
+Text GLabel 5350 3700 2    50   Input ~ 0
+CAP2
+Text GLabel 5350 3900 2    50   Input ~ 0
+CAP4
+Text GLabel 5350 3800 2    50   Input ~ 0
+CAP3
+Text GLabel 5350 4000 2    50   Input ~ 0
+io1
+Text GLabel 5350 4100 2    50   Input ~ 0
+io2
+Text GLabel 3350 4100 0    50   Input ~ 0
+io3
+Text GLabel 3350 4000 0    50   Input ~ 0
+io4
+Text GLabel 3350 3900 0    50   Input ~ 0
+io5
+Text GLabel 3350 3800 0    50   Input ~ 0
+io6
+NoConn ~ 3350 3700
+NoConn ~ 3350 3600
+NoConn ~ 3350 3500
+NoConn ~ 3350 3400
+NoConn ~ 3350 3300
+NoConn ~ 3350 3200
+NoConn ~ 3350 3100
+NoConn ~ 3350 3000
+NoConn ~ 3350 2900
+NoConn ~ 3350 2800
+NoConn ~ 3350 2700
+NoConn ~ 3350 2600
+NoConn ~ 3350 2500
+NoConn ~ 3350 2400
 $EndSCHEMATC

Commit message: nRF52 + ESP WROOM
Parts:
- added C?: 4.7uF, Capacitor_SMD:C_0402_1005Metric, symbol Device:C
- added C?: 0.1uF, Capacitor_SMD:C_0402_1005Metric, symbol Device:C
Connections:
- net +3V3: now also C?.1, C?.1
- net GND: now also C?.2, C?.2
Changed lines of the file:
@@
 $Descr A4 11693 8268
 encoding utf-8
-Sheet 3 8
+Sheet 3 9
 Title ""
 Date ""
@@
 NoConn ~ 3350 2500
 NoConn ~ 3350 2400
+$Comp
+L Device:C C?
+U 1 1 5E8C23CF
+P 1950 2050
+AR Path="/5E8C23CF" Ref="C?"  Part="1"
+AR Path="/5E4CCB9A/5E8C23CF" Ref="C?"  Part="1"
+F 0 "C?" H 2065 2096 50  0000 L CNN
+F 1 "4.7uF" H 2065 2005 50  0000 L CNN
+F 2 "Capacitor_SMD:C_0402_1005Metric" H 1988 1900 50  0001 C CNN
+F 3 "~" H 1950 2050 50  0001 C CNN
+	1    1950 2050
+	1    0    0    -1
+$EndComp
+$Comp
+L Device:C C?
+U 1 1 5E8C23D5
+P 2550 2050
+AR Path="/5E8C23D5" Ref="C?"  Part="1"
+AR Path="/5E4CCB9A/5E8C23D5" Ref="C?"  Part="1"
+F 0 "C?" H 2665 2096 50  0000 L CNN
+F 1 "0.1uF" H 2665 2005 50  0000 L CNN
+F 2 "Capacitor_SMD:C_0402_1005Metric" H 2588 1900 50  0001 C CNN
+F 3 "~" H 2550 2050 50  0001 C CNN
+	1    2550 2050
+	1    0    0    -1
+$EndComp
+$Comp
+L power:GND #PWR?
+U 1 1 5E8C23DB
+P 2250 2550
+AR Path="/5E8C23DB" Ref="#PWR?"  Part="1"
+AR Path="/5E4CCB9A/5E8C23DB" Ref="#PWR?"  Part="1"
+F 0 "#PWR?" H 2250 2300 50  0001 C CNN
+F 1 "GND" H 2255 2377 50  0000 C CNN
+F 2 "" H 2250 2550 50  0001 C CNN
+F 3 "" H 2250 2550 50  0001 C CNN
+	1    2250 2550
+	1    0    0    -1
+$EndComp
+$Comp
+L power:+3V3 #PWR?
+U 1 1 5E8C23E1
+P 2250 1650
+AR Path="/5E8C23E1" Ref="#PWR?"  Part="1"
+AR Path="/5E4CCB9A/5E8C23E1" Ref="#PWR?"  Part="1"
+F 0 "#PWR?" H 2250 1500 50  0001 C CNN
+F 1 "+3V3" H 2265 1823 50  0000 C CNN
+F 2 "" H 2250 1650 50  0001 C CNN
+F 3 "" H 2250 1650 50  0001 C CNN
+	1    2250 1650
+	1    0    0    -1
+$EndComp
+Wire Wire Line
+	1950 1900 1950 1750
+Wire Wire Line
+	1950 1750 2250 1750
+Wire Wire Line
+	2250 1750 2250 1650
+Wire Wire Line
+	2250 1750 2550 1750
+Wire Wire Line
+	2550 1750 2550 1900
+Connection ~ 2250 1750
+Wire Wire Line
+	1950 2200 1950 2400
+Wire Wire Line
+	1950 2400 2250 2400
+Wire Wire Line
+	2250 2400 2250 2550
+Wire Wire Line
+	2250 2400 2550 2400
+Wire Wire Line
+	2550 2400 2550 2200
+Connection ~ 2250 2400
 $EndSCHEMATC
